Commit message: 第七次提交
Co-Authored-By: Claude Opus 4.7 <noreply@anthropic.com>

File: src/wuyang_description/urdf/wuyang_arkermann.urdf.xacro (robot description, xacro)
@@ -1,3 +1,6 @@
 <?xml version="1.0"?>
+<!-- 宏定义：前轮转向系统 -->
+<xacro:macro name="front_steering_wheel" params="prefix y_reflect">
+</xacro:macro>
 <robot xmlns:xacro="http://www.ros.org/wiki/xacro" name="wuyang_arkermann">
     <!-- 定义颜色材质 -->

Commit message: 第八次提交
Co-Authored-By: Claude Opus 4.7 <noreply@anthropic.com>

File: src/wuyang_description/urdf/wuyang_arkermann.urdf.xacro (robot description, xacro)
@@ -24,5 +24,5 @@
             <origin xyz="0.0 0.0 0.0" rpy="0.0 0.0 0.0"/>
             <geometry>
-                <box size="4.8 1.76 2.16"/>
+                <box size="0.265 0.11 0.123"/>
             </geometry>
             <material name="sliver"/>
@@ -31,10 +31,10 @@
             <origin xyz="0.0 0.0 0.0" rpy="0.0 0.0 0.0"/>
             <geometry>
-                <box size="4.8 1.76 2.16"/>
+                <box size="0.265 0.11 0.123"/>
             </geometry>
         </collision>
     </link>
     <joint name="joint_name" type="fixed">
-        <origin xyz="0.0 0.0 1.12" rpy="0.0 0.0 0.0"/>
+        <origin xyz="0.0 0.0 0.0765" rpy="0.0 0.0 0.0"/>
         <parent link="base_footprint"/>
         <child link="base_link"/>
