Commit message: 5 times commit

File: src/wuyang_description/urdf/wuyang_arkermann.urdf.xacro (robot description, xacro)
@@ -21,5 +21,5 @@
             <origin xyz="0.0 0.0 0.0" rpy="0.0 0.0 0.0"/>
             <geometry>
-                <box size="0.0 0.0 0.0"/>
+                <box size="4.8 1.76 2.16"/>
             </geometry>
             <material name="">
@@ -31,5 +31,5 @@
             <origin xyz="0.0 0.0 0.0" rpy="0.0 0.0 0.0"/>
             <geometry>
-                <box size="0.0 0.0 0.0"/>
+                <box size="4.8 1.76 2.16"/>
             </geometry>
         </collision>

Commit message: the 6th commit

File: src/wuyang_description/urdf/wuyang_arkermann.urdf.xacro (robot description, xacro)
@@ -23,8 +23,5 @@
                 <box size="4.8 1.76 2.16"/>
             </geometry>
-            <material name="">
-                <color rgba="1.0 0.0 0.0 1.0"/>
-                <texture filename=""/>
-            </material>
+            <material name="sliver"/>
         </visual>
         <collision>
@@ -35,3 +32,10 @@
         </collision>
     </link>
+    <joint name="joint_name" type="fixed">
+        <origin xyz="0.0 0.0 1.12" rpy="0.0 0.0 0.0"/>
+        <parent link="base_footprint"/>
+        <child link="base_link"/>
+        <axis xyz="0.0 0.0 0.0"/>
+        <limit lower="0.0" upper="0.0" effort="0.0" velocity="0.0"/>
+    </joint>
 </robot>

Commit message: 第九次提交

File: src/wuyang_description/urdf/wuyang_arkermann.urdf.xacro (robot description, xacro)
@@ -1,6 +1,3 @@
 <?xml version="1.0"?>
-<!-- 宏定义：前轮转向系统 -->
-<xacro:macro name="front_steering_wheel" params="prefix y_reflect">
-</xacro:macro>
 <robot xmlns:xacro="http://www.ros.org/wiki/xacro" name="wuyang_arkermann">
     <!-- 定义颜色材质 -->
@@ -42,3 +39,53 @@
         <limit lower="0.0" upper="0.0" effort="0.0" velocity="0.0"/>
     </joint>
+    <!-- 宏定义：前轮转向系统 -->
+    <xacro:macro name="front_steering_wheel" params="prefix y_reflect">
+        <!-- 转向节（knuckle）：连接转向关节和滚动关节的中间连杆 -->
+        <link name="${prefix}_knuckle">
+            <inertial>
+                <origin xyz="0.0 0.0 0.0" rpy="0.0 0.0 0.0"/>
+                <mass value="0.05"/>
+                <inertia ixx="0.00001" ixy="0.0" ixz="0.0" iyy="0.00001" iyz="0.0" izz="0.00001"/>
+            </inertial>
+        </link>
+        <!-- 转向关节：base_link → 转向节，绕Z轴旋转实现转向 -->
+        <joint name="${prefix}_steering_joint" type="revolute">
+            <origin xyz="0.072 ${0.079 * y_reflect} -0.0425" rpy="0.0 0.0 0.0"/>
+            <parent link="base_link"/>
+            <child link="${prefix}_knuckle"/>
+            <axis xyz="0.0 0.0 1.0"/>
+            <limit lower="-0.6055" upper="0.6055" effort="10.0" velocity="10.0"/>
+        </joint>
+        <!-- 轮子 -->
+        <link name="${prefix}_wheel">
+            <inertial>
+                <origin xyz="0.0 0.0 0.0" rpy="0.0 0.0 0.0"/>
+                <mass value="0.1"/>
+                <inertia ixx="0.0001" ixy="0.0" ixz="0.0" iyy="0.0001" iyz="0.0" izz="0.0001"/>
+            </inertial>
+            <visual>
+                <origin xyz="0.0 0.0 0.0" rpy="1.5708 0.0 0.0"/>
+                <geometry>
+                    <cylinder radius="0.034" length="0.026"/>
+                </geometry>
+                <material name="black"/>
+            </visual>
+            <collision>
+                <origin xyz="0.0 0.0 0.0" rpy="1.5708 0.0 0.0"/>
+                <geometry>
+                    <cylinder radius="0.034" length="0.026"/>
+                </geometry>
+            </collision>
+        </link>
+        <!-- 滚动关节：转向节 → 轮子，绕Y轴连续旋转 -->
+        <joint name="${prefix}_rolling_joint" type="continuous">
+            <origin xyz="0.0 0.0 0.0" rpy="0.0 0.0 0.0"/>
+            <parent link="${prefix}_knuckle"/>
+            <child link="${prefix}_wheel"/>
+            <axis xyz="0.0 1.0 0.0"/>
+        </joint>
+    </xacro:macro>
+    <!-- 实例化左右前轮 -->
+    <xacro:front_steering_wheel prefix="left_front" y_reflect="1"/>
+    <xacro:front_steering_wheel prefix="right_front" y_reflect="-1"/>
 </robot>

Commit message: 第十次提交

File: src/wuyang_description/urdf/wuyang_arkermann.urdf.xacro (robot description, xacro)
@@ -15,6 +15,6 @@
         <inertial>
             <origin xyz="0.0 0.0 0.0" rpy="0.0 0.0 0.0"/>
-            <mass value="0.0"/>
-            <inertia ixx="0.0" ixy="0.0" ixz="0.0" iyy="0.0" iyz="0.0" izz="0.0"/>
+            <mass value="3.0"/>
+            <inertia ixx="0.0068" ixy="0.0" ixz="0.0" iyy="0.0213" iyz="0.0" izz="0.0206"/>
         </inertial>
         <visual name="RectangularPrism">
@@ -45,6 +45,6 @@
             <inertial>
                 <origin xyz="0.0 0.0 0.0" rpy="0.0 0.0 0.0"/>
-                <mass value="0.05"/>
-                <inertia ixx="0.00001" ixy="0.0" ixz="0.0" iyy="0.00001" iyz="0.0" izz="0.00001"/>
+                <mass value="0.0"/>
+                <inertia ixx="0.0000" ixy="0.0" ixz="0.0" iyy="0.0000" iyz="0.0" izz="0.0000"/>
             </inertial>
         </link>

Commit message: 第十一次提交

File: src/wuyang_description/urdf/wuyang_arkermann.urdf.xacro (robot description, xacro)
@@ -86,6 +86,38 @@
         </joint>
     </xacro:macro>
+    <!-- 宏定义：后轮（无转向，仅滚动） -->
+    <xacro:macro name="rear_wheel" params="prefix y_reflect">
+        <link name="${prefix}_wheel">
+            <inertial>
+                <origin xyz="0.0 0.0 0.0" rpy="0.0 0.0 0.0"/>
+                <mass value="0.1"/>
+                <inertia ixx="0.0001" ixy="0.0" ixz="0.0" iyy="0.0001" iyz="0.0" izz="0.0001"/>
+            </inertial>
+            <visual>
+                <origin xyz="0.0 0.0 0.0" rpy="1.5708 0.0 0.0"/>
+                <geometry>
+                    <cylinder radius="0.034" length="0.026"/>
+                </geometry>
+                <material name="black"/>
+            </visual>
+            <collision>
+                <origin xyz="0.0 0.0 0.0" rpy="1.5708 0.0 0.0"/>
+                <geometry>
+                    <cylinder radius="0.034" length="0.026"/>
+                </geometry>
+            </collision>
+        </link>
+        <joint name="${prefix}_rolling_joint" type="continuous">
+            <origin xyz="-0.072 ${0.079 * y_reflect} -0.0425" rpy="0.0 0.0 0.0"/>
+            <parent link="base_link"/>
+            <child link="${prefix}_wheel"/>
+            <axis xyz="0.0 1.0 0.0"/>
+        </joint>
+    </xacro:macro>
     <!-- 实例化左右前轮 -->
     <xacro:front_steering_wheel prefix="left_front" y_reflect="1"/>
     <xacro:front_steering_wheel prefix="right_front" y_reflect="-1"/>
+    <!-- 实例化左右后轮 -->
+    <xacro:rear_wheel prefix="left_rear" y_reflect="1"/>
+    <xacro:rear_wheel prefix="right_rear" y_reflect="-1"/>
 </robot>
