Commit message: 第十七次提交

File: src/wuyang_description/urdf/gazebo_control.urdf.xacro (robot description, xacro)
@@ -22,4 +22,10 @@
         </joint>
     </xacro:macro>
+    <xacro:macro name="front_rolling_interface" params="prefix">
+        <joint name="${prefix}_rolling_joint">
+            <state_interface name="velocity"/>
+            <state_interface name="position"/>
+        </joint>
+    </xacro:macro>
     <!-- 主宏：gazebo_control -->
     <xacro:macro name="gazebo_control" params="">

Commit message: 第十九次提交,修复了/joint_states话题为空的BUG

File: src/wuyang_description/urdf/gazebo_control.urdf.xacro (robot description, xacro)
@@ -31,5 +31,5 @@
     <!-- Camera pitch interface macro: non-controlled, used to get camera pose from gazebo -->
     <xacro:macro name="camera_pitch">
-        <joint name="camera_mount_joint">
+        <joint name="camera_base_joint">
             <state_interface name="position"/>
             <state_interface name="velocity"/>

File: src/wuyang_description/urdf/sensor_camera.urdf.xacro (robot description, xacro)
@@ -28,5 +28,5 @@
                 <origin xyz="0.0 0.0 0.0" rpy="0.0 0.0 0.0"/>
                 <mass value="0.1"/>
-                <inertia ixx="0.0001" ixy="0.0" ixz="0.0" iyy="0.00001" iyz="0.0" izz="0.00001"/>
+                <inertia ixx="0.00001" ixy="0.0" ixz="0.0" iyy="0.00001" iyz="0.0" izz="0.00001"/>
             </inertial>
         </link>

Commit message: 第二十次提交

File: src/wuyang_description/urdf/gazebo_control.urdf.xacro (robot description, xacro)
@@ -37,5 +37,5 @@
     </xacro:macro>
     <!-- Main macro: gazebo_control -->
-    <xacro:macro name="gazebo_control" params="">
+    <xacro:macro name="gazebo_control">
         <ros2_control name="GazeboSystem" type="system">
             <hardware>

File: src/wuyang_description/urdf/sensor_camera.urdf.xacro (robot description, xacro)
@@ -46,4 +46,29 @@
             <axis xyz="0.0 0.0 0.0"/>
         </joint>
+        <gazebo reference="camera_body_link">
+            <sensor type="depth" name="camera_sensor">
+                <plugin name="depth_camera" filename="libgazebo_ros_camera.so">
+                    <frame_name>camera_optical_link</frame_name>
+                </plugin>
+                <always_on>true</always_on>
+                <update_rate>10</update_rate>
+                <camera name="camera">
+                    <horizontal_fov>1.5009831567</horizontal_fov>
+                </camera>
+                <image>
+                    <width>800</width>
+                    <height>600</height>
+                    <format>R8G8B8</format>
+                </image>
+                <distortion>
+                    <k1>0.0</k1>
+                    <k2>0.0</k2>
+                    <k3>0.0</k3>
+                    <p1>0.0</p1>
+                    <p2>0.0</p2>
+                    <center>0.5 0.5</center>
+                </distortion>
+            </sensor>
+        </gazebo>
     </xacro:macro>
 </robot>

File: src/wuyang_description/urdf/sensor_laser.urdf.xacro (robot description, xacro)
@@ -1,5 +1,5 @@
 <?xml version="1.0"?>
 <robot xmlns:xacro="http://www.ros.org/wiki/xacro" name="sensor_laser">
-    <xacro:macro name="LS_p10m" params="parent xyz">
+    <xacro:macro name="LS_m10p" params="parent xyz">
         <link name="laser_link">
             <inertial>
@@ -28,4 +28,42 @@
             <axis xyz="0.0 0.0 0.0"/>
         </joint>
+        <gazebo reference="laser_link">
+            <sensor name="laserscan" type="ray">
+                <plugin name="laserscan" filename="libgazebo_ros_ray_sensor.so">
+                    <ros>
+                        <namespace>/</namespace>
+                        <remapping>~/out:=scan</remapping>
+                    </ros>
+                    <output_type>sensor_msgs/LaserScan</output_type>
+                    <frame_name>laser_link</frame_name>
+                </plugin>
+                <always_on>true</always_on>
+                <visualize>false</visualize>
+                <update_rate>5</update_rate>
+                <pose>0 0 0 0 0 0</pose>
+                <!-- 激光传感器配置 -->
+                <ray>
+                    <!-- 设置扫描角度范围 -->
+                    <scan>
+                        <horizontal>
+                            <samples>1500</samples>
+                            <resolution>1.000000</resolution>
+                            <min_angle>0.000000</min_angle>
+                            <max_angle>6.280000</max_angle>
+                        </horizontal>
+                    </scan>
+                    <range>
+                        <min>0.120000</min>
+                        <max>10.0</max>
+                        <resolution>0.015000</resolution>
+                    </range>
+                    <noise>
+                        <type>gaussian</type>
+                        <mean>0.0</mean>
+                        <stddev>0.01</stddev>
+                    </noise>
+                </ray>
+            </sensor>
+        </gazebo>
     </xacro:macro>
 </robot>

File: src/wuyang_description/urdf/wuyang_ackermann.urdf.xacro (robot description, xacro)
@@ -125,5 +125,5 @@
     <xacro:rear_wheel prefix="right_rear" y_reflect="-1"/>
     <!-- Instantiate LiDAR -->
-    <xacro:LS_p10m parent="base_link" xyz="0.059 0.0 0.109"/>
+    <xacro:LS_m10p parent="base_link" xyz="0.059 0.0 0.109"/>
     <!-- Instantiate camera: camera_pitch_link aligns with front top edge of chassis -->
     <xacro:GeminiPro_camera parent="base_link" xyz="0.1325 0.0 0.0615"/>
