Commit message: 第十八次提交,BUG:/joint_state话题为空

File: src/wuyang_description/urdf/full.urdf (robot description, URDF)
Before this commit: robot wuyang_ackermann, 11 links, 10 joints
Links:
- link camera_pitch_link: mass 0.0 -> 0.1
- link left_front_knuckle: mass 0.0 -> 0.1
- link right_front_knuckle: mass 0.0 -> 0.1

File: src/wuyang_description/urdf/gazebo_control.urdf.xacro (robot description, xacro)
@@ -1,5 +1,5 @@
 <?xml version="1.0"?>
 <robot xmlns:xacro="http://www.ros.org/wiki/xacro" name="gazebo_control">
-    <!-- 后轮控制接口宏：滚动速度控制 -->
+    <!-- Rear wheel control interface macro: rolling velocity control -->
     <xacro:macro name="rear_control_interface" params="prefix">
         <joint name="${prefix}_rolling_joint">
@@ -12,5 +12,5 @@
         </joint>
     </xacro:macro>
-    <!-- 前轮控制接口宏：转向角度控制 -->
+    <!-- Front wheel control interface macro: steering angle control -->
     <xacro:macro name="front_control_interface" params="prefix">
         <joint name="${prefix}_steering_joint">
@@ -22,4 +22,5 @@
         </joint>
     </xacro:macro>
+    <!-- Front wheel rolling interface macro: non-controlled, used to get front wheel pose from gazebo -->
     <xacro:macro name="front_rolling_interface" params="prefix">
         <joint name="${prefix}_rolling_joint">
@@ -28,5 +29,12 @@
         </joint>
     </xacro:macro>
-    <!-- 主宏：gazebo_control -->
+    <!-- Camera pitch interface macro: non-controlled, used to get camera pose from gazebo -->
+    <xacro:macro name="camera_pitch">
+        <joint name="camera_mount_joint">
+            <state_interface name="position"/>
+            <state_interface name="velocity"/>
+        </joint>
+    </xacro:macro>
+    <!-- Main macro: gazebo_control -->
     <xacro:macro name="gazebo_control" params="">
         <ros2_control name="GazeboSystem" type="system">
@@ -38,4 +46,7 @@
             <xacro:front_control_interface prefix="left_front"/>
             <xacro:front_control_interface prefix="right_front"/>
+            <xacro:front_rolling_interface prefix="left_front"/>
+            <xacro:front_rolling_interface prefix="right_front"/>
+            <xacro:camera_pitch/>
         </ros2_control>
         <gazebo>

File: src/wuyang_description/urdf/sensor_camera.urdf.xacro (robot description, xacro)
@@ -2,5 +2,5 @@
 <robot xmlns:xacro="http://www.ros.org/wiki/xacro" name="sensor_camera">
     <xacro:macro name="GeminiPro_camera" params="parent xyz">
-        <!-- 摄像头本体：黑色长方体 11.5cm x 1.7cm x 2.2cm -->
+        <!-- Camera body: black rectangular prism 11.5cm x 1.7cm x 2.2cm -->
         <link name="camera_body_link">
             <inertial>
@@ -23,13 +23,13 @@
             </collision>
         </link>
-        <!-- 相机俯仰link，无实体 -->
+        <!-- Camera pitch link -->
         <link name="camera_pitch_link">
             <inertial>
                 <origin xyz="0.0 0.0 0.0" rpy="0.0 0.0 0.0"/>
-                <mass value="0.0"/>
-                <inertia ixx="0.0" ixy="0.0" ixz="0.0" iyy="0.0" iyz="0.0" izz="0.0"/>
+                <mass value="0.1"/>
+                <inertia ixx="0.0001" ixy="0.0" ixz="0.0" iyy="0.00001" iyz="0.0" izz="0.00001"/>
             </inertial>
         </link>
-        <!-- Revolute joint: parent → camera_pitch_link，绕Y轴旋转0~45度（向前俯仰） -->
+        <!-- Revolute joint: parent → camera_pitch_link, rotates around Y axis 0~45 degrees (forward pitch) -->
         <joint name="camera_base_joint" type="revolute">
             <origin xyz="${xyz}" rpy="0.0 0.0 0.0"/>

File: src/wuyang_description/urdf/wuyang_ackermann.urdf.xacro (robot description, xacro)
@@ -4,5 +4,5 @@
     <xacro:include filename="sensor_camera.urdf.xacro"/>
     <xacro:include filename="gazebo_control.urdf.xacro"/>
-    <!-- 定义颜色材质 -->
+    <!-- Define color materials -->
     <material name="black">
         <color rgba="0.0 0.0 0.0 1.0" />
@@ -42,15 +42,15 @@
         <limit lower="0.0" upper="0.0" effort="0.0" velocity="0.0"/>
     </joint>
-    <!-- 宏定义：前轮转向系统 -->
+    <!-- Macro: front wheel steering system -->
     <xacro:macro name="front_steering_wheel" params="prefix y_reflect">
-        <!-- 转向节（knuckle）：连接转向关节和滚动关节的中间连杆 -->
+        <!-- Steering knuckle: intermediate link connecting steering joint and rolling joint -->
         <link name="${prefix}_knuckle">
             <inertial>
                 <origin xyz="0.0 0.0 0.0" rpy="0.0 0.0 0.0"/>
-                <mass value="0.0"/>
-                <inertia ixx="0.0000" ixy="0.0" ixz="0.0" iyy="0.0000" iyz="0.0" izz="0.0000"/>
+                <mass value="0.1"/>
+                <inertia ixx="0.00001" ixy="0.0" ixz="0.0" iyy="0.00001" iyz="0.0" izz="0.00001"/>
             </inertial>
         </link>
-        <!-- 转向关节：base_link → 转向节，绕Z轴旋转实现转向 -->
+        <!-- Steering joint: base_link → knuckle, rotates around Z axis for steering -->
         <joint name="${prefix}_steering_joint" type="revolute">
             <origin xyz="0.072 ${0.079 * y_reflect} -0.0425" rpy="0.0 0.0 0.0"/>
@@ -60,5 +60,5 @@
             <limit lower="-0.6055" upper="0.6055" effort="10.0" velocity="10.0"/>
         </joint>
-        <!-- 轮子 -->
+        <!-- Wheel -->
         <link name="${prefix}_wheel">
             <inertial>
@@ -81,5 +81,5 @@
             </collision>
         </link>
-        <!-- 滚动关节：转向节 → 轮子，绕Y轴连续旋转 -->
+        <!-- Rolling joint: knuckle → wheel, continuous rotation around Y axis -->
         <joint name="${prefix}_rolling_joint" type="continuous">
             <origin xyz="0.0 0.0 0.0" rpy="0.0 0.0 0.0"/>
@@ -89,5 +89,5 @@
         </joint>
     </xacro:macro>
-    <!-- 宏定义：后轮（无转向，仅滚动） -->
+    <!-- Macro: rear wheel (no steering, rolling only) -->
     <xacro:macro name="rear_wheel" params="prefix y_reflect">
         <link name="${prefix}_wheel">
@@ -118,15 +118,15 @@
         </joint>
     </xacro:macro>
-    <!-- 实例化左右前轮 -->
+    <!-- Instantiate left and right front wheels -->
     <xacro:front_steering_wheel prefix="left_front" y_reflect="1"/>
     <xacro:front_steering_wheel prefix="right_front" y_reflect="-1"/>
-    <!-- 实例化左右后轮 -->
+    <!-- Instantiate left and right rear wheels -->
     <xacro:rear_wheel prefix="left_rear" y_reflect="1"/>
     <xacro:rear_wheel prefix="right_rear" y_reflect="-1"/>
-    <!-- 实例化激光雷达 -->
+    <!-- Instantiate LiDAR -->
     <xacro:LS_p10m parent="base_link" xyz="0.059 0.0 0.109"/>
-    <!-- 实例化摄像头：camera_pitch_link 与车身前上方棱重合 -->
+    <!-- Instantiate camera: camera_pitch_link aligns with front top edge of chassis -->
     <xacro:GeminiPro_camera parent="base_link" xyz="0.1325 0.0 0.0615"/>
-    <!-- 实例化gazebo_control：包含ros2_control接口和gazebo插件 -->
+    <!-- Instantiate gazebo_control: includes ros2_control interfaces and gazebo plugin -->
     <xacro:gazebo_control/>
 </robot>

Commit message: 第二十次提交,完成雷达和摄像头硬件仿真

File: src/wuyang_description/urdf/full.urdf (robot description, URDF)
Before this commit: robot wuyang_ackermann, 11 links, 10 joints
Links:
- added link camera_optical_link
Joints:
- added joint camera_optical_joint: type fixed, parent camera_body_link, child camera_optical_link, origin xyz=0 0 0 rpy=-1.5708 0 -1.5708

File: src/wuyang_description/urdf/gazebo_control.urdf.xacro (robot description, xacro)
@@ -1,5 +1,4 @@
 <?xml version="1.0"?>
 <robot xmlns:xacro="http://www.ros.org/wiki/xacro" name="gazebo_control">
-    <!-- Rear wheel control interface macro: rolling velocity control -->
     <xacro:macro name="rear_control_interface" params="prefix">
         <joint name="${prefix}_rolling_joint">
@@ -12,5 +11,4 @@
         </joint>
     </xacro:macro>
-    <!-- Front wheel control interface macro: steering angle control -->
     <xacro:macro name="front_control_interface" params="prefix">
         <joint name="${prefix}_steering_joint">
@@ -22,5 +20,4 @@
         </joint>
     </xacro:macro>
-    <!-- Front wheel rolling interface macro: non-controlled, used to get front wheel pose from gazebo -->
     <xacro:macro name="front_rolling_interface" params="prefix">
         <joint name="${prefix}_rolling_joint">
@@ -29,5 +26,4 @@
         </joint>
     </xacro:macro>
-    <!-- Camera pitch interface macro: non-controlled, used to get camera pose from gazebo -->
     <xacro:macro name="camera_pitch">
         <joint name="camera_base_joint">
@@ -36,5 +32,4 @@
         </joint>
     </xacro:macro>
-    <!-- Main macro: gazebo_control -->
     <xacro:macro name="gazebo_control">
         <ros2_control name="GazeboSystem" type="system">

File: src/wuyang_description/urdf/sensor_camera.urdf.xacro (robot description, xacro)
@@ -2,5 +2,4 @@
 <robot xmlns:xacro="http://www.ros.org/wiki/xacro" name="sensor_camera">
     <xacro:macro name="GeminiPro_camera" params="parent xyz">
-        <!-- Camera body: black rectangular prism 11.5cm x 1.7cm x 2.2cm -->
         <link name="camera_body_link">
             <inertial>
@@ -23,5 +22,4 @@
             </collision>
         </link>
-        <!-- Camera pitch link -->
         <link name="camera_pitch_link">
             <inertial>
@@ -31,5 +29,4 @@
             </inertial>
         </link>
-        <!-- Revolute joint: parent → camera_pitch_link, rotates around Y axis 0~45 degrees (forward pitch) -->
         <joint name="camera_base_joint" type="revolute">
             <origin xyz="${xyz}" rpy="0.0 0.0 0.0"/>
@@ -39,5 +36,4 @@
             <limit lower="0.0" upper="0.7854" effort="1.0" velocity="1.0"/>
         </joint>
-        <!-- Fixed joint: camera_pitch_link → camera_body_link -->
         <joint name="camera_mount_joint" type="fixed">
             <origin xyz="-0.0085 0.0 0.011" rpy="0.0 0.0 0.0"/>
@@ -46,27 +42,45 @@
             <axis xyz="0.0 0.0 0.0"/>
         </joint>
+        <link name="camera_optical_link"/>
+        <joint name="camera_optical_joint" type="fixed">
+            <origin xyz="0 0 0" rpy="-1.5708 0 -1.5708"/>
+            <parent link="camera_body_link"/>
+            <child link="camera_optical_link"/>
+        </joint>
         <gazebo reference="camera_body_link">
-            <sensor type="depth" name="camera_sensor">
-                <plugin name="depth_camera" filename="libgazebo_ros_camera.so">
+            <sensor type="depth" name="gemini_pro_sensor">
+                <always_on>true</always_on>
+                <update_rate>30.0</update_rate>
+                <camera name="camera">
+                    <horizontal_fov>1.5708</horizontal_fov>
+                    <image>
+                        <width>800</width>
+                        <height>600</height>
+                        <format>R8G8B8</format>
+                    </image>
+                    <clip>
+                        <near>0.15</near>
+                        <far>10.0</far>
+                    </clip>
+                    <noise>
+                        <type>gaussian</type>
+                        <mean>0.0</mean>
+                        <stddev>0.007</stddev>
+                    </noise>
+                </camera>
+                <plugin name="gemini_camera_controller" filename="libgazebo_ros_camera.so">
+                    <ros>
+                        <namespace></namespace>
+                        <remapping>~/image_raw:=image_raw</remapping>
+                        <remapping>~/camera_info:=camera_info</remapping>
+                        <remapping>~/depth/image_raw:=depth/image_raw</remapping>
+                        <remapping>~/depth/camera_info:=depth/camera_info</remapping>
+                        <remapping>~/points:=points</remapping>
+                    </ros>
+                    <camera_name>gemini_pro</camera_name>
                     <frame_name>camera_optical_link</frame_name>
+                    <min_depth>0.15</min_depth>
+                    <max_depth>10.0</max_depth>
                 </plugin>
-                <always_on>true</always_on>
-                <update_rate>10</update_rate>
-                <camera name="camera">
-                    <horizontal_fov>1.5009831567</horizontal_fov>
-                </camera>
-                <image>
-                    <width>800</width>
-                    <height>600</height>
-                    <format>R8G8B8</format>
-                </image>
-                <distortion>
-                    <k1>0.0</k1>
-                    <k2>0.0</k2>
-                    <k3>0.0</k3>
-                    <p1>0.0</p1>
-                    <p2>0.0</p2>
-                    <center>0.5 0.5</center>
-                </distortion>
             </sensor>
         </gazebo>

File: src/wuyang_description/urdf/sensor_laser.urdf.xacro (robot description, xacro)
@@ -42,7 +42,5 @@
                 <update_rate>5</update_rate>
                 <pose>0 0 0 0 0 0</pose>
-                <!-- 激光传感器配置 -->
                 <ray>
-                    <!-- 设置扫描角度范围 -->
                     <scan>
                         <horizontal>

File: src/wuyang_description/urdf/wuyang_ackermann.urdf.xacro (robot description, xacro)
@@ -4,5 +4,4 @@
     <xacro:include filename="sensor_camera.urdf.xacro"/>
     <xacro:include filename="gazebo_control.urdf.xacro"/>
-    <!-- Define color materials -->
     <material name="black">
         <color rgba="0.0 0.0 0.0 1.0" />
@@ -42,7 +41,5 @@
         <limit lower="0.0" upper="0.0" effort="0.0" velocity="0.0"/>
     </joint>
-    <!-- Macro: front wheel steering system -->
     <xacro:macro name="front_steering_wheel" params="prefix y_reflect">
-        <!-- Steering knuckle: intermediate link connecting steering joint and rolling joint -->
         <link name="${prefix}_knuckle">
             <inertial>
@@ -52,5 +49,4 @@
             </inertial>
         </link>
-        <!-- Steering joint: base_link → knuckle, rotates around Z axis for steering -->
         <joint name="${prefix}_steering_joint" type="revolute">
             <origin xyz="0.072 ${0.079 * y_reflect} -0.0425" rpy="0.0 0.0 0.0"/>
@@ -60,5 +56,4 @@
             <limit lower="-0.6055" upper="0.6055" effort="10.0" velocity="10.0"/>
         </joint>
-        <!-- Wheel -->
         <link name="${prefix}_wheel">
             <inertial>
@@ -81,5 +76,4 @@
             </collision>
         </link>
-        <!-- Rolling joint: knuckle → wheel, continuous rotation around Y axis -->
         <joint name="${prefix}_rolling_joint" type="continuous">
             <origin xyz="0.0 0.0 0.0" rpy="0.0 0.0 0.0"/>
@@ -89,5 +83,4 @@
         </joint>
     </xacro:macro>
-    <!-- Macro: rear wheel (no steering, rolling only) -->
     <xacro:macro name="rear_wheel" params="prefix y_reflect">
         <link name="${prefix}_wheel">
@@ -118,15 +111,10 @@
         </joint>
     </xacro:macro>
-    <!-- Instantiate left and right front wheels -->
     <xacro:front_steering_wheel prefix="left_front" y_reflect="1"/>
     <xacro:front_steering_wheel prefix="right_front" y_reflect="-1"/>
-    <!-- Instantiate left and right rear wheels -->
     <xacro:rear_wheel prefix="left_rear" y_reflect="1"/>
     <xacro:rear_wheel prefix="right_rear" y_reflect="-1"/>
-    <!-- Instantiate LiDAR -->
     <xacro:LS_m10p parent="base_link" xyz="0.059 0.0 0.109"/>
-    <!-- Instantiate camera: camera_pitch_link aligns with front top edge of chassis -->
     <xacro:GeminiPro_camera parent="base_link" xyz="0.1325 0.0 0.0615"/>
-    <!-- Instantiate gazebo_control: includes ros2_control interfaces and gazebo plugin -->
     <xacro:gazebo_control/>
 </robot>
