Commit message: feat: 添加 RTAB-Map 视觉 SLAM 支持
- config/rtabmap.yaml: RGB-D SLAM 参数配置
- launch/vslam.launch.py: 视觉 SLAM 启动文件
- package.xml: 添加 rtabmap_ros 依赖
- sensor_camera.urdf.xacro: 相机默认 25° 俯角

Co-Authored-By: Claude <noreply@anthropic.com>

File: src/wuyang_description/urdf/sensor_camera.urdf.xacro (robot description, xacro)
@@ -30,5 +30,5 @@
         </link>
         <joint name="camera_base_joint" type="revolute">
-            <origin xyz="${xyz}" rpy="0.0 0.0 0.0"/>
+            <origin xyz="${xyz}" rpy="0.0 0.4363 0.0"/>
             <parent link="${parent}"/>
             <child link="camera_pitch_link"/>

Commit message: revert: 取消摄像头 25° 俯角，恢复水平朝向
Co-Authored-By: Claude <noreply@anthropic.com>

File: src/wuyang_description/urdf/sensor_camera.urdf.xacro (robot description, xacro)
@@ -30,5 +30,5 @@
         </link>
         <joint name="camera_base_joint" type="revolute">
-            <origin xyz="${xyz}" rpy="0.0 0.4363 0.0"/>
+            <origin xyz="${xyz}" rpy="0.0 0.0 0.0"/>
             <parent link="${parent}"/>
             <child link="camera_pitch_link"/>
