Commit message: 第十三次提交

File: install/wuyang_description/share/wuyang_description/urdf/sensor_camera.urdf.xacro (robot description, xacro)
@@ -23,13 +23,5 @@
             </collision>
         </link>
-        <!-- 前下方俯仰转向link，无实体 -->
-        <link name="front_lower_pitch">
-            <inertial>
-                <origin xyz="0.0 0.0 0.0" rpy="0.0 0.0 0.0"/>
-                <mass value="0.0"/>
-                <inertia ixx="0.0" ixy="0.0" ixz="0.0" iyy="0.0" iyz="0.0" izz="0.0"/>
-            </inertial>
-        </link>
-        <!-- 相机安装连接link，无实体 -->
+        <!-- 相机俯仰link，无实体 -->
         <link name="camera_pitch_link">
             <inertial>
@@ -39,24 +31,17 @@
             </inertial>
         </link>
-        <!-- Revolute joint: camera_pitch_link → front_lower_pitch，绕Y轴旋转0~45度（向前俯仰） -->
-        <joint name="camera_pitch_joint" type="revolute">
-            <origin xyz="0.0 0.0 0.0" rpy="0.0 0.0 0.0"/>
-            <parent link="camera_pitch_link"/>
-            <child link="front_lower_pitch"/>
+        <!-- Revolute joint: parent → camera_pitch_link，绕Y轴旋转0~45度（向前俯仰） -->
+        <joint name="camera_base_joint" type="revolute">
+            <origin xyz="${xyz}" rpy="0.0 0.0 0.0"/>
+            <parent link="${parent}"/>
+            <child link="camera_pitch_link"/>
             <axis xyz="0.0 1.0 0.0"/>
             <limit lower="0.0" upper="0.7854" effort="1.0" velocity="1.0"/>
         </joint>
-        <!-- Fixed joint: front_lower_pitch → camera_body_link，摄像头前下棱与front_lower_pitch重合 -->
+        <!-- Fixed joint: camera_pitch_link → camera_body_link -->
         <joint name="camera_mount_joint" type="fixed">
             <origin xyz="-0.0085 0.0 0.011" rpy="0.0 0.0 0.0"/>
-            <parent link="front_lower_pitch"/>
+            <parent link="camera_pitch_link"/>
             <child link="camera_body_link"/>
-            <axis xyz="0.0 0.0 0.0"/>
-        </joint>
-        <!-- Fixed joint: parent → camera_pitch_link -->
-        <joint name="camera_base_joint" type="fixed">
-            <origin xyz="${xyz}" rpy="0.0 0.0 0.0"/>
-            <parent link="${parent}"/>
-            <child link="camera_pitch_link"/>
             <axis xyz="0.0 0.0 0.0"/>
         </joint>
